File: Electronics/BatCapMeter/BatCapMeter.kicad_pcb (KiCad board)
At the start: 2 copper layers, 200.4 x 75 mm, 28 parts, among them J1 5V Power, J2 BatteryHolder, J3 R_PROG, J4 B0 Conn, J5 B0 Conn, J6 B1 Conn, J7 B2 Conn, J8 B3 Conn, Q1 SI2301CDS, Q2 SI2302DDS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

Commit message: Prep for release v0.7.0
Parts:
- added D2: Discharge, LED_THT:LED_D3.0mm_Clear, F.Cu at (200.5, 139.5)
- added J10: Fan, Connector_PinHeader_2.54mm:PinHeader_1x02_P2.54mm_Horizontal, F.Cu at (204.0, 139.9)
- added J9: ExtBattery, Connector_JST:JST_PH_S2B-PH-K_1x02_P2.00mm_Horizontal, F.Cu at (249.4, 114.0)
- added Q5: SI2302DDS, Package_TO_SOT_SMD:SOT-23, B.Cu at (187.3, 139.3)
- added R9: 5.1k, Resistor_SMD:R_1206_3216Metric_Pad1.30x1.75mm_HandSolder, B.Cu at (193.5, 138.0)
- D1: value Power Ind -> Power; footprint LED_THT:LED_D3.0mm -> LED_THT:LED_D3.0mm_Clear
- J5: value B0 Conn -> BCM Conn
- moved D1 1.37 mm to (180.5, 141.0)
Routing:
- net /BC_O+B_V: track 64.6 -> 138.1 mm
- net /BC_DCH_CTL: track 25.4 -> 71.8 mm, vias 2 -> 4
- net /BC_+5V: track 31.9 -> 70.2 mm, vias 0 -> 2
- net Net-(J10-Pin_1): track 0.00 -> 19.7 mm
- net GND1: track 160.6 -> 174.0 mm
- net Net-(BO1-B-): track 124.6 -> 137.0 mm, vias 0 -> 1
- net Net-(D2-A): track 0.00 -> 3.53 mm
- net /BC_CH_C: track 29.7 -> 33.1 mm
- net (no net): vias 16 -> 15
Other:
- outline, holes or cut-outs redrawn
- board text added: "+ -"
- board text added: "Lipo Capacity Meter Controller v1.1.0"
- board text removed: "Lipo Capacity Meter Controller v1.0.0"

Commit message: Release v0.8.0
Parts:
- added JP1: Calib, Connector_PinHeader_2.54mm:PinHeader_1x02_P2.54mm_Vertical, F.Cu at (165.0, 111.1)
Connections:
- J2 pad 2: /BC_O+B_V -> Net-(J2-Pin_2)
- J9 pad 2: /BC_O+B_V -> Net-(J2-Pin_2)
Routing:
- net /BC_O+B_V: track 138.1 -> 35.5 mm
- net Net-(J2-Pin_2): track 0.00 -> 99.9 mm
Other:
- board text added: "${PROJ_NAME} Controller v${VERSION}"
- board text added: "${PROJ_NAME} Host v${VERSION}"
- board text removed: "Lipo Capacity Meter Controller v1.1.0"
- board text removed: "Lipo Capacity Meter Host v1.0.0"
