File: Electronics/BatCapMeter/BatCapMeter.kicad_sch (KiCad schematic)
At the start: 28 parts, among them J1 5V Power, J2 BatteryHolder, J3 R_PROG, J4 B0 Conn, J5 B0 Conn, J6 B1 Conn, J7 B2 Conn, J8 B3 Conn, Q1 SI2301CDS, Q2 SI2302DDS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

Commit message: Change to managing by State Machine
Other:
- title: (none) -> Battery Capacity Meter II
Changed lines of the file:
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@@
 	(generator_version "8.0")
 	(paper "A4")
+	(title_block
+		(title "Battery Capacity Meter II")
+		(rev "v0.1")
+	)
 	(junction
 		(at 72.39 30.48)

Commit message: Prep for release v0.7.0
Parts:
- added D2: Discharge, LED_THT:LED_D3.0mm_Clear, symbol Device:LED
- added J10: Fan, Connector_PinHeader_2.54mm:PinHeader_1x02_P2.54mm_Horizontal, symbol Connector:Conn_01x02_Socket
- added J9: ExtBattery, Connector_JST:JST_PH_S2B-PH-K_1x02_P2.00mm_Horizontal, symbol Connector:Conn_01x02_Socket
- added Q5: SI2302DDS, Package_TO_SOT_SMD:SOT-23, symbol Device:Q_NMOS_GSD
- added R9: 5.1k, Resistor_SMD:R_1206_3216Metric_Pad1.30x1.75mm_HandSolder, symbol Device:R_US
- D1: value Power Ind -> Power; footprint LED_THT:LED_D3.0mm -> LED_THT:LED_D3.0mm_Clear
- J5: value B0 Conn -> BCM Conn
Connections:
- net BC_+5V: now also J10.2 (Pin_2)
- net BC_DCH_CTL: now also Q5.1 (G), R9.1
- net BC_O+B_V: now also J9.2 (Pin_2)
- net GND1: now also D2.1 (K), Q5.2 (S)
- net at BO1.4 (B-), J2.1 (Pin_1): now also J9.1 (Pin_1)
- new net: D2.2 (A), R9.2
- new net: J10.1 (Pin_1), Q5.3 (D)
Other:
- moved on the sheet: R3

Commit message: Release v0.8.0
Parts:
- added JP1: Calib, Connector_PinHeader_2.54mm:PinHeader_1x02_P2.54mm_Vertical, symbol Jumper:Jumper_2_Small_Bridged
Connections:
- net BC_O+B_V: now also JP1.1 (A); no longer J2.2 (Pin_2), J9.2 (Pin_2)
- new net: J2.2 (Pin_2), J9.2 (Pin_2), JP1.2 (B)
Other:
- title: Battery Capacity Meter II -> ${PROJ_NAME}
Changed lines of the file:
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@@
 	(paper "A4")
 	(title_block
-		(title "Battery Capacity Meter II")
-		(rev "v0.1")
+		(title "${PROJ_NAME}")
+		(date "2025-05-04")
+		(rev "${VERSION}")
 	)
 	(rectangle
@@
 	(wire
 		(pts
-			(xy 91.44 149.86) (xy 91.44 167.64)
+			(xy 91.44 149.86) (xy 91.44 154.94)
 		)
 		(stroke
@@
 	(wire
 		(pts
+			(xy 91.44 160.02) (xy 91.44 167.64)
+		)
+		(stroke
+			(width 0)
+			(type default)
+		)
+	)
+	(wire
+		(pts
 			(xy 181.61 83.82) (xy 181.61 90.17)
 		)
@@
 					(unit 1)
 				)
+			)
+		)
+	)
+	(symbol
+		(lib_id "Jumper:Jumper_2_Small_Bridged")
+		(at 91.44 157.48 270)
+		(unit 1)
+		(exclude_from_sim yes)
+		(in_bom yes)
+		(on_board yes)
+		(dnp no)
+		(fields_autoplaced yes)
+		(property "Reference" "JP1"
+			(at 92.71 156.2099 90)
+			(effects
+				(font
+					(size 1.27 1.27)
+				)
+				(justify left)
+			)
+		)
+		(property "Value" "Calib"
+			(at 92.71 158.7499 90)
+			(effects
+				(font
+					(size 1.27 1.27)
+				)
+				(justify left)
+			)
+		)
+		(property "Footprint" "Connector_PinHeader_2.54mm:PinHeader_1x02_P2.54mm_Vertical"
+			(at 91.44 157.48 0)
+			(effects
+				(font
+					(size 1.27 1.27)
+				)
+				(hide yes)
+			)
+		)
+		(property "Datasheet" "~"
+			(at 91.44 157.48 0)
+			(effects
+				(font
+					(size 1.27 1.27)
+				)
+				(hide yes)
+			)
+		)
+		(property "Description" "Jumper, 2-pole, small symbol, bridged"
+			(at 91.44 157.48 0)
+			(effects
+				(font
+					(size 1.27 1.27)
+				)
+				(hide yes)
+			)
+		)
+		(pin "1"
+		)
+		(pin "2"
+		)
+		(instances
+			(project ""
+				(path "/d838ee05-8219-4637-8a5b-7a554bf6dff8"
+					(reference "JP1")
+					(unit 1)
+				)

Commit message: Prep for Release 0.9.0
Parts:
- BO1, D1, D2, J10, J2, J3, J5, J9, JP1, Q1, Q2, Q3, Q4, Q5, R1, R2, R3, R5, R7, R8, R9: Board (none) -> BC
- BO2, BO3, BO4, J1, J4, J6, J7, J8, OLED1, R4, R6, U1, U2: Board (none) -> Master
